File: KicadJE_Face.kicad_pcb (KiCad board)
At the start: 2 copper layers, 242 x 128 mm, 39 parts

Commit message: Update KicadJE_Face.kicad_pcb
Parts:
- removed the G*** at (175.0, 156.8)
- removed the G*** at (11.0, 161.0)
- removed the H101 at (11.0, 51.0)
- removed the H102 at (171.5, 39.0)
- removed the H102 at (-2.50, 39.0)
- removed the H103 at (171.5, 161.0)
- removed the H103 at (-2.50, 161.0)
- removed the H104 at (24.5, 39.0)
- removed the H105 at (24.5, 161.0)
- removed H301: ON, AJ:LED_Hole_3mm
- removed the TP102 at (1.00, 115.0)
- removed the TP103 at (21.0, 125.0)
- removed the TP105 at (21.0, 145.0)
- removed the TP106 at (1.08, 145.0)
- removed the TP107 at (21.0, 84.5)
- removed the TP107 at (21.0, 115.0)
- removed the TP107 at (21.0, 65.0)
- removed the TP108 at (1.00, 125.0)
- removed the TP112 at (1.00, 84.5)
- removed the TP112 at (1.00, 65.0)
- removed TP301: In1, AJ:Jack_6m3
- removed TP302: Tri, AJ:Jack_6m3
- removed TP303: SQ, AJ:Jack_6m3
- removed TP304: PWM1, AJ:Pot_6m3_scale1
- removed TP305: PWM2, AJ:Pot_6m3_scale1
- moved TP107 31.0 mm to (223.0, 96.0)
- moved TP112 31.0 mm to (203.0, 96.0)
Other:
- board size 242 x 128 mm -> 40 x 128 mm
- board text added: "Johansen Engineering OLED Rev A 12/04-2021"
- board text added: "MOD 1"
- board text added: "MOD 2"
- board text added: "OLED"
- board text removed: "CV"
- board text removed: "CV Util Rev A 22/03-2020 Johansen Engineering"
- board text removed: "GLIDE"
- board text removed: "Gain1"
- board text removed: "Gain2"
- board text removed: "Glide1"
- board text removed: "Glide2"
- board text removed: "IN"
- board text removed: "Inv1"
- board text removed: "Inv2"
- board text removed: "Johansen Engineering Glide Rev A 22/03-2020"
- board text removed: "Offset1"
- board text removed: "Offset2"
- board text removed: "Phase1"
- board text removed: "Phase2"
- board text removed: "SHIFT"
- board text removed: "TIME"
- board text removed: "TimeShift Rev A 22/03-2020 Johansen Engineering"
